File: dmxdude.kicad_sch (KiCad schematic)
At the start: 0 parts

Commit message: power circuitry
Other:
- added sheet Power (power.kicad_sch)
Changed lines of the file:
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@@
+	)
+	(sheet
+		(at 193.04 48.26)
+		(size 22.86 16.51)
+		(exclude_from_sim no)
+		(in_bom yes)
+		(on_board yes)
+		(dnp no)
+		(fields_autoplaced yes)
+		(stroke
+			(width 0.1524)
+			(type solid)
+		)
+		(fill
+			(color 0 0 0 0.0000)
+		)
+		(property "Sheetname" "Power"
+			(at 193.04 47.5484 0)
+			(effects
+				(font
+					(size 1.27 1.27)
+				)
+				(justify left bottom)
+			)
+		)
+		(property "Sheetfile" "power.kicad_sch"
+			(at 193.04 65.3546 0)
+			(effects
+				(font
+					(size 1.27 1.27)
+				)
+				(justify left top)
+			)
+		)
+		(instances
+			(project "dmxdude"
+				(path "/bd7590c0-6a37-4bf0-a9f2-f26180744ceb"
+					(page "5")
+				)
+			)
+		)
 	)
 	(sheet
