File: dmxdude.kicad_pcb (KiCad board)
At the start: 2 copper layers, 61 x 81.3 mm, 91 parts, among them J1 NC3MAAH, J10 Screw_Terminal_01x02, J11 USB_C_Receptacle_USB2.0_16P, J12 Screw_Terminal_01x03, J2 NC3FAAH, J3 MSD-11-A, J4 Screw_Terminal_01x03, J5 Screw_Terminal_01x02, J6 Screw_Terminal_01x02, J7 Screw_Terminal_01x02, J8 Screw_Terminal_01x02, J9 Screw_Terminal_01x02, Q1 IRLZ44N, Q2 IRLZ44N, Q3 IRLZ44N, Q4 IRLZ44N, Q5 IRLZ44N, Q6 IRLZ44N, U1 ST485E, U2 74AHCT125, U3 74AHCT125, U4 ESP32-S3-WROOM-1, U5 STM32C011F4Ux, Y1 Crystal_GND24

Commit message: power circuitry
Parts:
- added C16: 100n, Capacitor_SMD:C_0603_1608Metric_Pad1.08x0.95mm_HandSolder, F.Cu at (80.3, 128.2)
- added C17: 100n, Capacitor_SMD:C_0603_1608Metric_Pad1.08x0.95mm_HandSolder, F.Cu at (58.0, 118.4)
- added C18: C_Polarized, Capacitor_THT:CP_Radial_D5.0mm_P2.00mm, F.Cu at (76.7, 134.1)
- added C19: 1u, Capacitor_SMD:C_0603_1608Metric_Pad1.08x0.95mm_HandSolder, F.Cu at (58.0, 120.9)
- added C20: 10u, Capacitor_SMD:C_0805_2012Metric_Pad1.18x1.45mm_HandSolder, F.Cu at (91.4, 124.5)
- added C21: 10u, Capacitor_SMD:C_0805_2012Metric_Pad1.18x1.45mm_HandSolder, F.Cu at (91.4, 121.9)
- added C22: 1u, Capacitor_SMD:C_0603_1608Metric_Pad1.08x0.95mm_HandSolder, F.Cu at (58.0, 123.4)
- added C23: 1u, Capacitor_SMD:C_0603_1608Metric_Pad1.08x0.95mm_HandSolder, F.Cu at (58.0, 125.9)
- added D12: LED, LED_SMD:LED_0603_1608Metric_Pad1.05x0.95mm_HandSolder, F.Cu at (66.7, 137.7)
- added J13: Screw_Terminal_01x02, TerminalBlock_MetzConnect:TerminalBlock_MetzConnect_Type101_RT01602HBWC_1x02_P5.08mm_Horizontal, F.Cu at (114.3, 110.6)
- added L1: SRR1050A-270Y, SamacSys_Parts:SRR1050A221Y, F.Cu at (87.9, 132.1)
- added R32: 100k, Resistor_SMD:R_0603_1608Metric_Pad0.98x0.95mm_HandSolder, F.Cu at (76.7, 123.5)
- added R33: 19.1k, Resistor_SMD:R_0603_1608Metric_Pad0.98x0.95mm_HandSolder, F.Cu at (74.7, 125.6)
- added R34: 470, Resistor_SMD:R_0603_1608Metric_Pad0.98x0.95mm_HandSolder, F.Cu at (58.0, 133.4)
- added U6: LM66100DCK, Package_TO_SOT_SMD:SOT-363_SC-70-6, F.Cu at (98.0, 126.5)
- added U7: LM66100DCK, Package_TO_SOT_SMD:SOT-363_SC-70-6, F.Cu at (98.0, 122.9)
- added U8: LMR51610XDBVR, SamacSys_Parts:SOT95P280X145-6N, F.Cu at (77.7, 128.0)
- added U9: TLV74033PDBVR, SamacSys_Parts:SOT95P280X145-5N, F.Cu at (70.1, 113.8)
Connections:
- J11 pad A4: Net-(D12-A) -> VBUS
- J11 pad A9: Net-(D12-A) -> VBUS
- J11 pad B4: Net-(D12-A) -> VBUS
- J11 pad B9: Net-(D12-A) -> VBUS
Other:
- board outline removed

Commit message: add probe headers
Parts:
- removed the D12 at (129.8, 62.2)
- added J1: Conn_01x04, Connector_PinHeader_2.54mm:PinHeader_1x04_P2.54mm_Vertical, F.Cu at (63.8, 149.9)
- added J15: Conn_01x04, Connector_PinHeader_2.54mm:PinHeader_1x04_P2.54mm_Vertical, F.Cu at (63.8, 135.7)
- added J_ESP_1: Conn_01x04, Connector_PinHeader_2.54mm:PinHeader_1x04_P2.54mm_Vertical, F.Cu at (52.6, 135.7)
- added J_ESP_2: Conn_01x05, Connector_PinSocket_2.54mm:PinSocket_1x05_P2.54mm_Vertical, F.Cu at (48.0, 135.7)
- added J_SD1: Conn_01x04, Connector_PinHeader_2.54mm:PinHeader_1x04_P2.54mm_Vertical, F.Cu at (57.2, 135.7)
- added J_STM1: Conn_01x09, Connector_PinHeader_2.54mm:PinHeader_1x09_P2.54mm_Vertical, F.Cu at (211.8, 93.7)
- *R1: footprint Resistor_SMD:R_0201_0603Metric_Pad0.64x0.40mm_HandSolder -> Resistor_SMD:R_0603_1608Metric_Pad0.98x0.95mm_HandSolder
- moved C17 216.1 mm to (273.1, 142.8)
- moved C18 216.1 mm to (273.1, 140.3)
- moved C22 216.1 mm to (273.1, 145.3)
- moved C23 216.1 mm to (273.1, 147.8)
- moved R34 209.8 mm to (267.1, 151.7)
- moved D13 209.8 mm to (275.7, 156.0)
- moved C3 197.3 mm to (253.2, 98.6)
- moved C4 197.3 mm to (253.2, 101.1)
- moved U9 190.6 mm to (258.1, 145.3)
- moved R25 171.1 mm to (261.5, 110.2)
- moved R24 171.0 mm to (257.0, 107.7)
- moved C8 163.2 mm to (245.3, 99.4)
- moved U7 160.7 mm to (258.1, 137.2)
- moved U8 160.7 mm to (258.1, 140.7)
- moved C16 160.7 mm to (236.7, 148.3)
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- renumbered *C4 to *C1, *C3 to *C2, C11 to C10, C8 to C11, C9 to C12, C7 to C13, C13 to C14, C12 to C15, C18 to C16, C19 to C17, C17 to C18, C16 to C19, C14 to C3, C15 to C4, C6 to C5, C5 to C6, C3 to C7, C4 to C8, C10 to C9, D13 to D1, D9 to D11, D11 to D12, D12 to D13, D1 to D9, J12 to J10, J4 to J11, J11 to J12, J3 to J13, J13 to J14, J1 to J2, J2 to J3, J5 to J4, J6 to J5, J7 to J6, J8 to J7, J9 to J8, J10 to J9, R2 to R1, R9 to R10, R10 to R11, R11 to R12, R12 to R13, R13 to R14, R14 to R15, R17 to R16, R1 to R17, R21 to R19, R3 to R2, R23 to R20, R20 to R21, R19 to R22, R16 to R23, R15 to R24, R24 to R25, R25 to R26, R26 to R27, R27 to R28, R28 to R29, R22 to R3, R29 to R30, R30 to R31, R8 to R4, R7 to R5, R5 to R7, R4 to R8, R31 to R9, S2 to S1, S1 to S2, U3 to U2, U2 to U3, U8 to U6, U6 to U8
Connections:
- net Net-(U4-IO46) renamed /MCU/J_ESP_2_2
- J2 pad G: unconnected-(J1-PadG) -> GND
- U4 pad 15: unconnected-(U4-IO3-Pad15) -> /MCU/J_ESP_2_1
- U4 pad 19: unconnected-(U4-IO11-Pad19) -> /MCU/J_ESP_2_5
- U4 pad 36: unconnected-(U4-RXD0-Pad36) -> /MCU/J_ESP_1_4
- U4 pad 37: unconnected-(U4-TXD0-Pad37) -> /MCU/J_ESP_1_3
- U4 pad 38: unconnected-(U4-IO2-Pad38) -> /MCU/J_ESP_1_2
- U4 pad 39: unconnected-(U4-IO1-Pad39) -> /MCU/J_ESP_1_1
- U5 pad 10: unconnected-(U5-PA5-Pad10) -> Net-(J_STM1-Pin_2)
- U5 pad 11: unconnected-(U5-PA6-Pad11) -> Net-(J_STM1-Pin_3)
- U5 pad 12: unconnected-(U5-PA7-Pad12) -> Net-(J_STM1-Pin_4)
- U5 pad 13: unconnected-(U5-PA8-Pad13) -> Net-(J_STM1-Pin_5)
- U5 pad 14: unconnected-(U5-PA9/PA11-Pad14) -> Net-(J_STM1-Pin_6)
- U5 pad 15: unconnected-(U5-PA10/PA12-Pad15) -> Net-(J_STM1-Pin_7)
Routing:
- net STM32_SWDCLK: track 0.00 -> 12.0 mm
- net Net-(J_STM1-Pin_2): track 0.00 -> 9.99 mm
- net STM32_SWDIO: track 0.00 -> 9.84 mm
- net Net-(J_STM1-Pin_7): track 0.00 -> 8.34 mm
- net Net-(J_STM1-Pin_3): track 0.00 -> 8.34 mm
- net Net-(J_STM1-Pin_6): track 0.00 -> 7.67 mm
- net Net-(J_STM1-Pin_4): track 0.00 -> 7.67 mm
- net Net-(J_STM1-Pin_5): track 0.00 -> 6.83 mm

Commit message: partial layout
Parts:
- removed TP1: TestPoint, Connector_PinHeader_2.54mm:PinHeader_1x01_P2.54mm_Vertical
- added C26: 100n, Capacitor_SMD:C_0603_1608Metric_Pad1.08x0.95mm_HandSolder, F.Cu at (239.0, 105.5)
- added D14: MM3Zxx, Diode_SMD:D_SOD-323F, F.Cu at (127.1, 155.7)
- added J16: Conn_02x04_Top_Bottom, Connector_PinHeader_2.54mm:PinHeader_2x04_P2.54mm_Vertical, F.Cu at (244.1, 131.1)
- added J_OLED_1: Conn_01x04, Connector_PinHeader_2.54mm:PinHeader_1x04_P2.54mm_Vertical, F.Cu at (240.8, 120.9)
- added R36: 100k, Resistor_SMD:R_0603_1608Metric_Pad0.98x0.95mm_HandSolder, F.Cu at (132.8, 154.0)
- added R37: 5.1k, Resistor_SMD:R_0603_1608Metric_Pad0.98x0.95mm_HandSolder, F.Cu at (132.6, 158.0)
- moved J15 228.1 mm to (291.3, 119.9), turned to 180 degrees
- moved J10 213.2 mm to (274.8, 95.5), turned to -90 degrees
- moved D1 205.6 mm to (252.1, 139.7)
- moved D3 205.6 mm to (252.1, 129.3)
- moved D4 205.6 mm to (252.1, 131.9)
- moved D5 205.6 mm to (252.1, 134.5)
- moved D6 205.6 mm to (252.1, 137.1)
- moved D2 205.5 mm to (252.1, 126.2)
- moved C5 200.3 mm to (59.7, 47.0), turned to 90 degrees
- moved C6 199.5 mm to (61.2, 47.0), turned to 90 degrees
- moved J1 193.8 mm to (252.0, 103.9)
- moved S1 192.7 mm to (253.2, 148.3), turned to 90 degrees
- moved J_ESP_2 192.6 mm to (237.2, 99.6), turned to -90 degrees
- moved S3 188.1 mm to (245.2, 53.0)
- moved S2 177.7 mm to (236.2, 148.3), turned to 90 degrees
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- renumbered C8 to C10, C9 to C11, C10 to C12, C11 to C13, C12 to C14, C13 to C15, C14 to C16, C15 to C17, C16 to C18, C17 to C19, C18 to C20, C19 to C21, C20 to C22, C21 to C23, C22 to C24, C23 to C25, *C1 to C3, *C2 to C4, C3 to C5, C4 to C6, C5 to C7, C6 to C8, C7 to C9, R9 to R10, R10 to R11, R11 to R12, R12 to R13, R13 to R14, R14 to R15, R15 to R16, R16 to R17, R17 to R18, R18 to R19, *R1 to R2, R19 to R20, R20 to R21, R21 to R22, R22 to R23, R23 to R24, R24 to R25, R25 to R26, R26 to R27, R27 to R28, R28 to R29, R2 to R3, R29 to R30, R30 to R31, R31 to R32, R32 to R33, R33 to R34, R34 to R35, R3 to R4, R4 to R5, R5 to R6, R6 to R7, R7 to R8, R8 to R9
Connections:
- net Net-(U4-USB_D+) renamed USB+
- net Net-(U4-USB_D-) renamed USB-
Routing:
- net ESP32_BOOT: track 0.00 -> 67.6 mm
- net DMX_TX: track 0.00 -> 46.8 mm
- net DMX_RX: track 0.00 -> 45.2 mm
- net DMX-: track 0.00 -> 43.2 mm
- net DMX+: track 0.00 -> 34.9 mm
- net STM32_TX: track 0.00 -> 22.8 mm
- net +5V: track 0.00 -> 21.6 mm
- net STM32_RX: track 0.00 -> 19.6 mm
- net OLED_SDA: track 0.00 -> 15.2 mm
- net DMX_DE: track 0.00 -> 12.4 mm
- net OLED_SCL: track 0.00 -> 12.2 mm
- net GND: track 0.00 -> 9.39 mm
- net Net-(U5-PC15): track 0.00 -> 8.27 mm
- net STM32_SWDCLK: track 12.0 -> 6.01 mm
- net Net-(J_STM1-Pin_2): track 9.99 -> 15.3 mm
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Other:
- board outline added: 76.2 x 76.2 mm
