File: ws2812_output.kicad_sch (KiCad schematic)
At the start: 6 parts, among them J13 Conn_01x01, J14 Screw_Terminal_01x03, U8 74AHCT1G125

Commit message: complete layout, routing, and silkscreen
Parts:
- renumbered C22 to C21, C23 to C22
Changed lines of the file:
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@@
 		(on_board yes)
 		(dnp no)
-		(property "Reference" "C22"
+		(property "Reference" "C21"
 			(at 113.03 59.69 90)
 			(effects
@@
 			(project "dmxdude-mini"
 				(path "/bd7590c0-6a37-4bf0-a9f2-f26180744ceb/337463c9-19f6-40f5-8e97-b16881129868/00e8db54-2aab-4140-b84c-fba32f59bb48"
-					(reference "C24")
-					(unit 1)
-				)
-				(path "/bd7590c0-6a37-4bf0-a9f2-f26180744ceb/337463c9-19f6-40f5-8e97-b16881129868/d3b8d2d5-c3e6-441a-bceb-837788c2901c"
-					(reference "C22")
+					(reference "C23")
+					(unit 1)
+				)
+				(path "/bd7590c0-6a37-4bf0-a9f2-f26180744ceb/337463c9-19f6-40f5-8e97-b16881129868/d3b8d2d5-c3e6-441a-bceb-837788c2901c"
+					(reference "C21")
 					(unit 1)
 				)
@@
 			(project "dmxdude-mini"
 				(path "/bd7590c0-6a37-4bf0-a9f2-f26180744ceb/337463c9-19f6-40f5-8e97-b16881129868/00e8db54-2aab-4140-b84c-fba32f59bb48"
-					(reference "D6")
+					(reference "RGB3")
 					(unit 1)
 				)
@@
 		(on_board yes)
 		(dnp no)
-		(property "Reference" "C23"
+		(property "Reference" "C22"
 			(at 125.73 114.3 90)
 			(effects
@@
 			(project "dmxdude-mini"
 				(path "/bd7590c0-6a37-4bf0-a9f2-f26180744ceb/337463c9-19f6-40f5-8e97-b16881129868/00e8db54-2aab-4140-b84c-fba32f59bb48"
-					(reference "C25")
-					(unit 1)
-				)
-				(path "/bd7590c0-6a37-4bf0-a9f2-f26180744ceb/337463c9-19f6-40f5-8e97-b16881129868/d3b8d2d5-c3e6-441a-bceb-837788c2901c"
-					(reference "C23")
-					(unit 1)
-				)
+					(reference "C24")
+					(unit 1)
+				)
+				(path "/bd7590c0-6a37-4bf0-a9f2-f26180744ceb/337463c9-19f6-40f5-8e97-b16881129868/d3b8d2d5-c3e6-441a-bceb-837788c2901c"
+					(reference "C22")
+					(unit 1)
+				)
