File: dmxdude-mini.kicad_pcb (KiCad board)
At the start: 2 copper layers, 63.5 x 76.2 mm, 87 parts, among them J1 Conn_01x04, J10 Screw_Terminal_01x03, J11 Screw_Terminal_01x03, J12 USB_C_Receptacle_USB2.0_16P, J13 MSD-11-A, J15 Conn_01x04, J2 NC3MAAH, J3 NC3FAAH, J4 Conn_01x08, J5 Conn_01x08, U1 ST485E, U2 74AHCT1G125, U3 74AHCT1G125, U4 ESP32-S3-WROOM-1, U5 STM32C011F4Ux, U6 LMR51610XDBVR, U7 LM66100DCK, U8 LM66100DCK, U9 TLV74033PDBVR, Y1 Crystal_GND24

Commit message: complete top layer layout
Parts:
- removed the C12 at (149.4, 44.9)
- removed the C5 at (101.1, 35.3)
- removed the C6 at (101.1, 37.8)
- removed the C7 at (55.4, 53.3)
- removed the C8 at (78.0, 53.6)
- removed D7, D8: WS2812B, LED_SMD:LED_WS2812B_PLCC4_5.0x5.0mm_P3.2mm
- removed the J10 at (54.7, 31.2)
- removed the J11 at (77.1, 31.2)
- removed J_STM1: Conn_01x09, Connector_PinHeader_2.54mm:PinHeader_1x09_P2.54mm_Vertical
- removed the U2 at (96.0, 36.1)
- removed the U3 at (96.0, 40.0)
- added C22: 100n, Capacitor_SMD:C_0603_1608Metric_Pad1.08x0.95mm_HandSolder, F.Cu at (147.2, 141.5)
- added C23: 100n, Capacitor_SMD:C_0603_1608Metric_Pad1.08x0.95mm_HandSolder, F.Cu at (138.7, 136.7)
- added C24: 100n, Capacitor_SMD:C_0603_1608Metric_Pad1.08x0.95mm_HandSolder, F.Cu at (164.2, 141.5)
- added C25: 100n, Capacitor_SMD:C_0603_1608Metric_Pad1.08x0.95mm_HandSolder, F.Cu at (155.7, 136.7)
- added D6: WS2812B, LED_SMD:LED_WS2812B_PLCC4_5.0x5.0mm_P3.2mm, F.Cu at (156.5, 140.5)
- added J13: Conn_01x01, Connector_PinHeader_2.54mm:PinHeader_1x01_P2.54mm_Vertical, F.Cu at (133.9, 137.7)
- added J14: Screw_Terminal_01x03, TerminalBlock_MetzConnect:TerminalBlock_MetzConnect_Type101_RT01603HBWC_1x03_P5.08mm_Horizontal, F.Cu at (134.9, 147.8)
- added J15: Conn_01x01, Connector_PinHeader_2.54mm:PinHeader_1x01_P2.54mm_Vertical, F.Cu at (150.9, 137.7)
- added J16: Screw_Terminal_01x03, TerminalBlock_MetzConnect:TerminalBlock_MetzConnect_Type101_RT01603HBWC_1x03_P5.08mm_Horizontal, F.Cu at (151.9, 147.8)
- added J4: Conn_01x01, Connector_PinHeader_2.54mm:PinHeader_1x01_P2.54mm_Vertical, F.Cu at (147.1, 133.9)
- added J5: Conn_01x10, Connector_PinHeader_2.54mm:PinHeader_1x10_P2.54mm_Vertical, F.Cu at (138.9, 99.6)
- added R5: 5.1k, Resistor_SMD:R_0603_1608Metric_Pad0.98x0.95mm_HandSolder, F.Cu at (184.9, 146.6)
- added RGB2: WS2812B, LED_SMD:LED_WS2812B_PLCC4_5.0x5.0mm_P3.2mm, F.Cu at (139.4, 140.5)
- added U8: 74AHCT1G125, Package_TO_SOT_SMD:SOT-353_SC-70-5_Handsoldering, F.Cu at (144.6, 140.7)
- added U9: 74AHCT1G125, Package_TO_SOT_SMD:SOT-353_SC-70-5_Handsoldering, F.Cu at (161.6, 140.7)
- J10: renamed from J13; moved to B.Cu
- moved D3 147.2 mm to (145.3, 114.8), turned to 180 degrees
- moved R17 145.0 mm to (145.3, 116.3), turned to 180 degrees
- moved R4 142.0 mm to (184.9, 143.0)
- moved RGB1 137.7 mm to (139.7, 114.3)
- moved C20 127.5 mm to (139.4, 132.6), turned to 180 degrees
- moved C10 127.1 mm to (135.9, 109.6), turned to 90 degrees
- moved D5 127.0 mm to (135.4, 127.5)
- moved C21 123.4 mm to (139.4, 126.0), turned to 180 degrees
- moved C18 122.3 mm to (145.8, 128.5), turned to 90 degrees
- moved R26 121.4 mm to (135.4, 129.3)
- moved C19 118.0 mm to (147.8, 128.5), turned to 90 degrees
- moved U6 115.9 mm to (143.0, 127.5), turned to 180 degrees
- moved U5 113.8 mm to (143.0, 131.1), turned to 180 degrees
- moved D4 110.8 mm to (158.0, 122.2), turned to 180 degrees
- moved R9 110.4 mm to (124.2, 102.4), turned to 180 degrees
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- renumbered C15 to C10, C16 to C11, C17 to C12, C18 to C13, C19 to C14, C20 to C15, C21 to C16, C26 to C17, C22 to C18, C23 to C19, C24 to C20, C25 to C21, C9 to C5, C10 to C6, C11 to C7, C13 to C8, C14 to C9, D9 to D1, D10 to D2, D11 to D3, D14 to D4, D13 to D5, J_SD1 to J11, J15 to J12, J4 to J6, J12 to J7, J5 to J8, J_OLED_1 to J9, R21 to R10, R22 to R11, R23 to R12, R24 to R13, R25 to R14, R26 to R15, R27 to R16, R28 to R17, R29 to R18, R30 to R19, R31 to R20, R32 to R21, R36 to R22, R37 to R23, R33 to R24, R34 to R25, R35 to R26, R17 to R6, R18 to R7, R19 to R8, R20 to R9, D12 to RGB1, U4 to U2, U5 to U3, U6 to U4, U7 to U5, U8 to U6, U9 to U7
Connections:
- J12 pad 2: +3.3V -> +VDC
- J12 pad 4: +VDC -> +3.3V
- J8 pad 1: /MCU/J_ESP_2_1 -> GND
- J8 pad 2: /MCU/J_ESP_2_2 -> +3.3V
- J8 pad 3: STM32_RX -> /MCU/J_ESP_2_1
- J8 pad 4: STM32_TX -> /MCU/J_ESP_2_2
- J8 pad 5: /MCU/J_ESP_2_5 -> STM32_RX
- J8 pad 6: /MCU/J_ESP_2_6 -> STM32_TX
- J8 pad 7: /MCU/J_ESP_2_7 -> /MCU/J_ESP_2_5
- J8 pad 8: unconnected-(J5-Pin_8-Pad8) -> /MCU/J_ESP_2_6
- RGB1 pad 4: ESP32_LED -> ESP32_WS2812
- U2 pad 19: /MCU/J_ESP_2_5 -> ESP32_WS2812
- U2 pad 21: /MCU/J_ESP_2_6 -> /MCU/J_ESP_2_5
- U2 pad 22: /MCU/J_ESP_2_7 -> /MCU/J_ESP_2_6
Routing:
- net DMX_RX: track 45.2 -> 11.9 mm
- net DMX_TX: track 46.8 -> 24.1 mm
- net OLED_SDA: track 15.2 -> 0.00 mm
- net OLED_SCL: track 12.2 -> 0.00 mm
- net +5V: track 15.0 -> 4.41 mm
- net Net-(U3-PC15): track 8.27 -> 2.07 mm
- net GND: track 9.39 -> 4.69 mm
- net DMX+: track 34.9 -> 38.9 mm
- net Net-(U3-PC14): track 5.34 -> 2.13 mm
- net V_SENSE_VDC: track 2.05 -> 0.07 mm
- net DMX-: track 43.2 -> 44.7 mm
Other:
- outline, holes or cut-outs redrawn
- board text added: "dmxdude mini"
- board text added: "v0 | June 2025 Cy Westbrook"

Commit message: complete layout, routing, and silkscreen
Parts:
- removed the C11 at (128.6, 30.7)
- C11: renamed from C12; moved to B.Cu
- J6, J8: footprint Connector_PinSocket_2.54mm:PinSocket_1x08_P2.54mm_Vertical -> Connector_PinHeader_2.54mm:PinHeader_1x08_P2.54mm_Vertical
- JP1, R4, R5: moved to B.Cu
- R18, R19, R20, R21: value 10k -> 470; moved to B.Cu
- moved R19 110.6 mm to (154.4, 131.3), turned to 180 degrees
- moved R21 107.5 mm to (154.4, 133.1), turned to 180 degrees
- moved R18 105.2 mm to (154.4, 126.0), turned to 180 degrees
- moved R20 104.8 mm to (154.4, 127.8), turned to 180 degrees
- moved C11 104.6 mm to (154.4, 129.5), turned to 180 degrees
- moved JP1 46.1 mm to (158.2, 106.4), turned to 180 degrees
- moved R5 41.3 mm to (147.1, 130.0), turned to 90 degrees
- moved R4 38.2 mm to (147.1, 137.7), turned to 90 degrees
- moved J2 26.7 mm to (156.7, 94.2)
- moved J3 26.4 mm to (122.7, 89.2)
- moved R8 25.6 mm to (133.3, 120.4), turned to 90 degrees
- moved C6 6.48 mm to (145.3, 108.7), turned to -90 degrees
- moved C5 5.97 mm to (139.2, 108.7), turned to 90 degrees
- moved R9 3.05 mm to (121.2, 102.4)
- moved R6 2.41 mm to (129.3, 141.7)
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- renumbered C13 to C12, C14 to C13, C15 to C14, C16 to C15, C17 to C16, C18 to C17, C19 to C18, C20 to C19, C21 to C20, C22 to C21, C23 to C22, C24 to C23, C25 to C24, D6 to RGB3
Connections:
- J10 pad P2: SD_CS -> Net-(J10-CD/DAT3)
- J10 pad P3: SD_MOSI -> Net-(J10-CMD)
- J10 pad P5: SD_SCK -> Net-(J10-CLK)
- J10 pad P7: SD_MISO -> Net-(J10-DAT0)
- R18 pad 1: +3.3V -> Net-(J10-DAT0)
- R18 pad 2: SD_CS -> SD_MISO
- R19 pad 1: +3.3V -> Net-(J10-CMD)
- R20 pad 1: +3.3V -> Net-(J10-CLK)
- R21 pad 1: +3.3V -> Net-(J10-CD/DAT3)
- R21 pad 2: SD_MISO -> SD_CS
- U2 pad 8: SD_MISO -> SD_SCK
- U2 pad 9: SD_SCK -> SD_MISO
Routing:
- net GND: track 4.69 -> 653.1 mm, vias 0 -> 25
- net +3.3V: track 3.25 -> 196.9 mm, vias 0 -> 5
- net OUT_EN: track 0.00 -> 102.1 mm
- net +5V: track 4.41 -> 104.5 mm, vias 0 -> 5
- net +VDC: track 0.00 -> 75.1 mm
- net SD_MOSI: track 0.00 -> 74.1 mm, vias 0 -> 1
- net SD_CS: track 0.00 -> 71.2 mm, vias 0 -> 1
- net WS2812_2: track 0.00 -> 66.4 mm, vias 0 -> 1
- net ESP32_BOOT: track 0.00 -> 59.6 mm
- net SD_MISO: track 0.00 -> 58.4 mm, vias 0 -> 1
- net SD_SCK: track 0.00 -> 58.4 mm, vias 0 -> 1
- net WS2812_1: track 0.00 -> 56.9 mm, vias 0 -> 1
- net USB+: track 0.00 -> 47.5 mm, vias 0 -> 2
- net USB-: track 0.00 -> 46.6 mm, vias 0 -> 2
- net DMX_DE: track 12.4 -> 55.6 mm, vias 0 -> 1
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- added copper zone on B.Cu, net GND
- added copper zone on F.Cu, net GND
- added copper zone on F.Cu, net Net-(U4-SW)
- added copper zone on F.Cu, net Net-(U5-~{CE})
Other:
- outline, holes or cut-outs redrawn
- board text added: "+3.3V"
- board text added: "+5V"
- board text added: "+VDC"
- board text added: "BOOT"
- board text added: "CS/IO6"
- board text added: "DMX_DE"
- board text added: "DMX_RE"
- board text added: "DMX_RX"
- board text added: "DMX_TX"
- board text added: "ESP32 EN"
- board text added: "GND"
- board text added: "IO1"
- board text added: "IO10/PB6"
- board text added: "IO13"
- board text added: "IO14"
- board text added: "IO2"
- board text added: "IO3"
- board text added: "IO39"
- board text added: "IO4/SCL"
- board text added: "IO40"
- board text added: "IO41"
- board text added: "IO42"
- board text added: "IO46"
- board text added: "IO5/SDA"
- board text added: "IO9/PB7"
- board text added: "MISO/IO16"
- board text added: "MOSI/IO7"
- board text added: "NRST"
- board text added: "OUT_EN"
- board text added: "PA10"
- board text added: "PA5"
- board text added: "PA6"
- board text added: "PA7"
- board text added: "PA8"
- board text added: "PA9"
- board text added: "RXD0"
- board text added: "SCK/IO15"
- board text added: "STM32 NRST"
- board text added: "SWDCLK"
- board text added: "SWDIO"
- board text added: "TXD0"
- board text added: "WS2812_1/IO21"
- board text added: "WS2812_2/IO47"

Commit message: final for order 23 june 2025
Other:
- board text added: "1/GND"
- board text added: "2/DMX-"
- board text added: "3/DMX+"
Changed lines of the file:
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@@
 		)
 	)
+	(gr_text "3/DMX+"
+		(at 152.908 92.71 0)
+		(layer "F.SilkS")
+		(effects
+			(font
+				(size 0.8 0.8)
+				(thickness 0.13)
+			)
+			(justify bottom)
+		)
+	)
+	(gr_text "1/GND"
+		(at 122.682 87.376 0)
+		(layer "F.SilkS")
+		(effects
+			(font
+				(size 0.8 0.8)
+				(thickness 0.13)
+			)
+			(justify bottom)
+		)
+	)
+	(gr_text "2/DMX-"
+		(at 130.302 87.884 0)
+		(layer "F.SilkS")
+		(effects
+			(font
+				(size 0.8 0.8)
+				(thickness 0.13)
+			)
+			(justify bottom)
+		)
+	)
 	(gr_text "ESP32 EN"
 		(at 108.966 127 90)
@@
 		)
 	)
+	(gr_text "GND"
+		(at 152.908 87.376 0)
+		(layer "F.SilkS")
+		(effects
+			(font
+				(size 0.8 0.8)
+				(thickness 0.13)
+			)
+			(justify bottom)
+		)
+	)
+	(gr_text "2/DMX-"
+		(at 149.098 91.186 0)
+		(layer "F.SilkS")
+		(effects
+			(font
+				(size 0.8 0.8)
+				(thickness 0.13)
+			)
+			(justify bottom)
+		)
+	)
 	(gr_text "BOOT"
 		(at 125.984 145.034 0)
@@
 		)
 	)
+	(gr_text "1/GND"
+		(at 156.718 91.186 0)
+		(layer "F.SilkS")
+		(effects
+			(font
+				(size 0.8 0.8)
+				(thickness 0.13)
+			)
+			(justify bottom)
+		)
+	)
+	(gr_text "3/DMX+"
+		(at 126.492 91.948 0)
+		(layer "F.SilkS")
+		(effects
+			(font
+				(size 0.8 0.8)
+				(thickness 0.13)
+			)
+			(justify bottom)
+		)
+	)
 	(gr_text "PA5"
 		(at 161.798 101.346 270)
@@
 		)
 	)
+	(gr_text "1/GND"
+		(at 122.682 87.376 0)
+		(layer "B.SilkS")
+		(effects
+			(font
+				(size 0.8 0.8)
+				(thickness 0.13)
+			)
+			(justify bottom mirror)
+		)
+	)
 	(gr_text "DMX_RX"
 		(at 152.908 104.013 0)
@@
 		)
 	)
+	(gr_text "2/DMX-"
+		(at 130.302 87.884 0)
+		(layer "B.SilkS")
+		(effects
+			(font
+				(size 0.8 0.8)
+				(thickness 0.13)
+			)
+			(justify bottom mirror)
+		)
+	)
 	(gr_text "GND"
 		(at 138.43 118.872 270)
@@
 		)
 	)
+	(gr_text "GND"
+		(at 152.908 87.376 0)
+		(layer "B.SilkS")
+		(effects
+			(font
+				(size 0.8 0.8)
+				(thickness 0.13)
+			)
+			(justify bottom mirror)
+		)
+	)
 	(gr_text "IO13"
 		(at 116.84 101.346 270)
@@
 		)
 	)
+	(gr_text "1/GND"
+		(at 156.718 91.186 0)
+		(layer "B.SilkS")
+		(effects
+			(font
+				(size 0.8 0.8)
+				(thickness 0.13)
+			)
+			(justify bottom mirror)
+		)
+	)
 	(gr_text "+3.3V"
 		(at 151.638 119.38 270)
@@
 		)
 	)
+	(gr_text "2/DMX-"
+		(at 149.098 91.186 0)
+		(layer "B.SilkS")
+		(effects
+			(font
+				(size 0.8 0.8)
+				(thickness 0.13)
+			)
+			(justify bottom mirror)
+		)
+	)
 	(gr_text "IO41"
 		(at 112.522 108.204 0)
@@
 		)
 	)
+	(gr_text "3/DMX+"
+		(at 126.492 91.948 0)
+		(layer "B.SilkS")
+		(effects
+			(font
+				(size 0.8 0.8)
+				(thickness 0.13)
+			)
+			(justify bottom mirror)
+		)
+	)
 	(gr_text "IO3"
 		(at 127 101.346 270)
@@
 		)
 	)
+	(gr_text "3/DMX+"
+		(at 152.908 92.71 0)
+		(layer "B.SilkS")
+		(effects
+			(font
+				(size 0.8 0.8)
+				(thickness 0.13)
+			)
+			(justify bottom mirror)
+		)
+	)
 	(segment
 		(start 151.892 147.828)
@@
 	)
 	(segment
-		(start 147.9795 127.335)
-		(end 152.989 127.335)
-		(width 0.3)
-		(layer "F.Cu")
-		(net 1)
-	)
-	(segment
 		(start 137.0565 128.524)
 		(end 136.2945 129.286)
@@
 	)
 	(segment
+		(start 147.828 127.4865)
+		(end 148.5685 126.746)
+		(width 0.3)
+		(layer "F.Cu")
+		(net 1)
+	)
+	(segment
 		(start 128.394 147.545)
 		(end 129.345 146.594)
@@
 	)
 	(segment
-		(start 147.828 127.4865)
-		(end 147.9795 127.335)
-		(width 0.3)
-		(layer "F.Cu")
-		(net 1)
-	)
-	(segment
 		(start 134.874 147.828)
 		(end 136.18 147.828)
@@
 	)
 	(segment
+		(start 148.5685 126.746)
+		(end 152.4 126.746)
+		(width 0.3)
+		(layer "F.Cu")
+		(net 1)
+	)
+	(segment
+		(start 152.4 126.746)
+		(end 154.432 128.778)
+		(width 0.3)
+		(layer "F.Cu")
+		(net 1)
+	)
+	(segment
 		(start 144.3755 116.9435)
 		(end 144.3755 116.332)
@@
 	)
 	(segment
-		(start 152.989 127.335)
-		(end 154.432 128.778)
-		(width 0.3)
-		(layer "F.Cu")
-		(net 1)
-	)
-	(segment
 		(start 162.052 102.108)
 		(end 161.155661 102.108)
@@
 	)
 	(segment
+		(start 161.697339 107.288661)
+		(end 162.957 107.288661)
+		(width 0.5)
+		(layer "F.Cu")
+		(net 4)
+	)
+	(segment
 		(start 165.608 140.9065)
 		(end 164.174 142.3405)
@@
 	)
 	(segment
-		(start 161.29 107.696)
-		(end 161.697339 107.288661)
-		(width 0.5)
-		(layer "F.Cu")
-		(net 4)
-	)
-	(segment
 		(start 141.224 130.81)
 		(end 140.97 130.556)
@@
 	)
 	(segment
-		(start 141.800266 125.984)
-		(end 141.224 126.560266)
-		(width 0.5)
-		(layer "F.Cu")
-		(net 4)
-	)
-	(segment
 		(start 141.596996 131.714)
 		(end 142.052 131.714)
@@
 	)
 	(segment
+		(start 141.800266 125.984)
+		(end 141.224 126.560266)
+		(width 0.5)
+		(layer "F.Cu")
+		(net 4)
+	)
+	(segment
 		(start 138.496 132.6065)
 		(end 138.5175 132.628)
@@
 	)
 	(segment
-		(start 141.595996 131.715)
-		(end 141.596996 131.714)
+		(start 154.178 117.729)
+		(end 145.923 125.984)
 		(width 0.5)
 		(layer "F.Cu")
@@
 	)
 	(segment
-		(start 161.29 110.49)
-		(end 161.29 107.696)
+		(start 141.595996 131.715)
+		(end 141.596996 131.714)
 		(width 0.5)
 		(layer "F.Cu")
@@
 	)
 	(segment
-		(start 141.224 126.560266)
-		(end 141.224 128.524)
-		(width 0.5)
-		(layer "F.Cu")
-		(net 4)
-	)
-	(segment
 		(start 161.51 103.478661)
 		(end 162.967339 103.478661)
@@
 	(segment
 		(start 154.178 117.602)
-		(end 145.796 125.984)
+		(end 154.432 117.602)
 		(width 0.5)
 		(layer "F.Cu")
@@
 	)
 	(segment
-		(start 161.697339 107.288661)
-		(end 162.957 107.288661)
+		(start 140.396 131.408)
+		(end 140.197 131.607)
 		(width 0.5)
 		(layer "F.Cu")
@@
 	)
 	(segment
-		(start 140.396 131.408)
-		(end 140.197 131.607)
+		(start 154.432 117.602)
+		(end 161.29 110.744)
 		(width 0.5)
 		(layer "F.Cu")
@@
 	)
 	(segment
-		(start 154.178 117.602)
-		(end 161.29 110.49)
+		(start 161.29 110.744)
+		(end 161.29 107.696)
 		(width 0.5)
 		(layer "F.Cu")
@@
 	)
 	(segment
+		(start 145.923 125.984)
+		(end 141.800266 125.984)
+		(width 0.5)
+		(layer "F.Cu")
+		(net 4)
+	)
+	(segment
 		(start 138.496 130.556)
 		(end 138.496 132.6065)
@@
 	)
 	(segment
-		(start 145.796 125.984)
-		(end 141.800266 125.984)
+		(start 141.224 126.560266)
+		(end 141.224 128.524)
+		(width 0.5)
+		(layer "F.Cu")
+		(net 4)
+	)
+	(segment
+		(start 154.178 117.602)
+		(end 154.178 117.729)
 		(width 0.5)
 		(layer "F.Cu")
@@
 	)
 	(segment
+		(start 161.29 107.696)
+		(end 161.697339 107.288661)
+		(width 0.5)
+		(layer "F.Cu")
+		(net 4)
+	)
+	(segment
 		(start 141.224 131.343004)
 		(end 141.224 130.81)
@@
 		(polygon
 			(pts
-				(xy 104.14 71.628) (xy 175.514 69.088) (xy 175.514 156.972) (xy 103.886 156.718)
+				(xy 102.87 71.12) (xy 176.53 71.12) (xy 176.53 154.94) (xy 102.87 154.94)
 			)
 		)
